File: kicad/stm8_platform/stepper.sch (KiCad schematic (older format))
At the start: 34 parts, among them J1 CONN_02X10, P1 UART, P2 SWIM, Q1 AO3401, Q2 AO3401, Q3 AO3401, SW1 SW_DIP_x03, U1 STM8S105K4T6C, U2 ULN2803A, U3 LD1117S50CTR

Commit message: +motherboard
Changed lines of the file:
@@
-EESchema Schematic File Version 4
+EESchema Schematic File Version 2
+LIBS:power
 LIBS:stepper-cache
-EELAYER 26 0
+EELAYER 25 0
 EELAYER END
 $Descr A4 11693 8268
@@
 Text Label 9650 2400 0    61   ~ 0
 GND
-Text Label 9650 2500 0    61   ~ 0
+Text Label 9700 2600 0    61   ~ 0
 RXD
-Text Label 9650 2600 0    61   ~ 0
+Text Label 9700 2500 0    61   ~ 0
 TXD
 $Comp
@@
 	1600 1400 1750 1400
 Wire Wire Line
-	1750 1500 1750 1600
+	1750 1600 1750 1500
 Wire Wire Line
 	1200 1700 1200 1600
 Wire Wire Line
-	1200 1600 1500 1600
+	1200 1600 1750 1600
 Connection ~ 800  1700
 Wire Wire Line
@@
 	1450 3650 1350 3650
 Wire Wire Line
-	1350 1800 1500 1800
+	1350 1800 1750 1800
 Wire Wire Line
 	1500 1800 1500 1600
@@
 	10650 2400 10650 2500
 Wire Wire Line
-	10100 3150 10300 3150
+	10100 3150 10700 3150
 Connection ~ 10300 3150
 Wire Wire Line
@@
 	10100 3650 10100 3950
 Wire Wire Line
-	10050 3950 10100 3950
-Wire Wire Line
-	10050 3850 10300 3850
-Wire Wire Line
-	10050 3750 10500 3750
+	10050 3950 10550 3950
+Wire Wire Line
+	10050 3850 10550 3850
+Wire Wire Line
+	10050 3750 10550 3750
 Wire Wire Line
 	10500 3750 10500 3650
@@
 	9400 3750 9450 3750
 Wire Wire Line
-	9450 3950 9400 3950
+	9400 3950 9450 3950
 Wire Wire Line
 	9450 3850 9400 3850
@@
 Connection ~ 9400 3750
 Wire Wire Line
-	9400 3950 9400 3850
+	9400 3650 9400 3950
 Wire Wire Line
 	1350 5100 1350 5150
 Wire Wire Line
-	1200 5650 1350 5650
+	1200 5650 1450 5650
 Wire Wire Line
 	2050 5650 1950 5650
@@
 	9250 1050 9250 1150
 Wire Wire Line
-	9750 1150 9850 1150
+	9750 1150 10700 1150
 Wire Wire Line
 	9850 1150 9850 1000
@@
 	8600 1250 8600 1150
 Wire Wire Line
-	7650 1150 7750 1150
-Wire Wire Line
-	8200 1600 8200 1550
-Wire Wire Line
-	7750 1550 8200 1550
+	7650 1150 7800 1150
+Wire Wire Line
+	8200 1450 8200 1600
+Wire Wire Line
+	7750 1550 8600 1550
 Connection ~ 8200 1550
 Connection ~ 7750 1150
@@
 	8150 2450 8350 2450
 Wire Wire Line
-	8250 2250 8250 2500
+	8250 2250 8250 2950
 Wire Wire Line
 	8250 2950 8600 2950
@@
 	850  3850 3100 3850
 Wire Wire Line
-	8100 5500 8200 5500
+	8100 5500 8600 5500
 Connection ~ 8200 5500
 Wire Wire Line
 	8050 4650 8050 4600
 Wire Wire Line
-	8050 4600 8200 4600
+	8050 4600 8600 4600
 Wire Notes Line
 	7350 3350 9100 3350
@@
 	3600 5100 3600 5150
 Wire Wire Line
-	3450 5650 3600 5650
+	3450 5650 3700 5650
 Connection ~ 3600 5650
 Wire Wire Line
@@
 	3600 3550 3600 3600
 Wire Wire Line
-	3450 4100 3600 4100
+	3450 4100 3700 4100
 Connection ~ 3600 4100
 Wire Wire Line
@@
 	5400 3300 850  3300
 Wire Wire Line
-	8150 2850 8450 2850
+	8150 2850 8500 2850
 Wire Wire Line
 	8450 2850 8450 2600
@@
 	8600 2650 8600 2700
 Wire Wire Line
-	8600 2650 8400 2650
-Wire Wire Line
-	8400 3150 8400 2650
+	8150 2650 8600 2650
+Wire Wire Line
+	8400 2650 8400 3150
 Connection ~ 8400 2650
 Connection ~ 8450 2850
 Wire Wire Line
-	8350 2400 8350 2450
+	8350 2400 8350 3050
+Text Label 9100 5500 0    61   ~ 0
+RXD
 Text Label 9100 5400 0    61   ~ 0
-RXD
-Text Label 9100 5500 0    61   ~ 0
 TXD
 $Comp
@@
 Connection ~ 8350 2450
 Wire Wire Line
-	8600 2500 8250 2500
+	8250 2500 8600 2500
 Connection ~ 8250 2500
 $Comp
@@
 $EndComp
 Wire Wire Line
-	800  1700 800  1850
-Wire Wire Line
-	1500 1600 1750 1600
-Wire Wire Line
-	1500 1800 1750 1800
-Wire Wire Line
-	10300 3150 10500 3150
-Wire Wire Line
-	10500 3750 10550 3750
-Wire Wire Line
-	10300 3850 10550 3850
-Wire Wire Line
-	10100 3950 10550 3950
-Wire Wire Line
-	9400 3850 9400 3750
-Wire Wire Line
-	10500 3150 10700 3150
-Wire Wire Line
-	9400 3750 9400 3650
-Wire Wire Line
-	1350 5650 1450 5650
-Wire Wire Line
-	9850 1150 10700 1150
-Wire Wire Line
-	8200 1550 8200 1450
-Wire Wire Line
-	8200 1550 8600 1550
-Wire Wire Line
-	7750 1150 7800 1150
-Wire Wire Line
-	8200 5500 8600 5500
-Wire Wire Line
-	3600 5650 3700 5650
-Wire Wire Line
-	3600 4100 3700 4100
-Wire Wire Line
-	8400 2650 8150 2650
-Wire Wire Line
-	8450 2850 8500 2850
-Wire Wire Line
-	8200 4600 8600 4600
-Wire Wire Line
-	8350 2450 8350 3050
-Wire Wire Line
-	8250 2500 8250 2950
-Wire Wire Line
-	800  1450 800  1700
+	800  1450 800  1850
 Wire Wire Line
 	4200 5650 4300 5650
