File: kicad/stm8_platform/stepper.kicad_pcb (KiCad board)
At the start: 2 copper layers, 45 x 51 mm, 32 parts, among them J1 CONN_02X10, P1 UART, P2 SWIM, Q1 AO3401, Q2 AO3401, Q3 AO3401, SW1 SW_DIP_x03, U1 STM8S105K4T6C, U2 ULN2803A, U3 LD1117S50CTR

Commit message: small update
Parts:
- added HOLE1: HOLE, modules:hole_3mm, F.Cu at (98.5, 74.0)
- added HOLE2: HOLE, modules:hole_3mm, F.Cu at (137.5, 74.0)
Routing:
- net GND: track 120.3 -> 219.0 mm, vias 5 -> 8
- net /PD4: track 45.1 -> 51.9 mm
- net +5V: track 259.7 -> 253.1 mm
- net /SWIM/PD1: track 49.9 -> 51.7 mm
- net /PB0: track 23.8 -> 25.3 mm
- net Net-(C1-Pad2): track 3.94 -> 2.60 mm
- net /PB1: track 23.4 -> 24.7 mm
- net /PD0: track 36.4 -> 35.1 mm
- net /PC2: track 30.7 -> 31.8 mm
- net /PD2: track 30.5 -> 31.5 mm
- net /PB2: track 22.5 -> 23.5 mm
- net /PD6: track 45.3 -> 46.0 mm
- net /PD7: track 35.2 -> 34.6 mm
- net /NRST: track 39.8 -> 40.4 mm
Other:
- net class 1: via_dia 1.5 -> 2
- net class Default: via_dia 0.6 -> 1.5; via_drill 0.4 -> 0.6

Commit message: add code for STM8-based 2stepper management board
Parts:
- P2: footprint Pin_Headers.pretty:Pin_Header_Angled_1x04_Pitch2.54mm -> Connector_PinHeader_2.54mm.pretty:PinHeader_1x03_P2.54mm_Horizontal
